Commit message: Fix xacro arg handling for ros2_control params

File: robot_arm_pick_place/colcon_ws/src/arm_description/urdf/arm.urdf.xacro (robot description, xacro)
@@ -2,5 +2,5 @@
 <robot name="simple_arm" xmlns:xacro="http://www.ros.org/wiki/xacro">
   <xacro:arg name="ros2_control_params" default=""/>
-  <xacro:property name="pi" value="3.141592653589793"/>
+  <xacro:property name="ros2_control_params" value="$(arg ros2_control_params)"/>
   <material name="gray">
     <color rgba="0.6 0.6 0.6 1.0"/>

Commit message: Fix xacro ros2_control param substitution

File: robot_arm_pick_place/colcon_ws/src/arm_description/urdf/arm.urdf.xacro (robot description, xacro)
@@ -2,5 +2,4 @@
 <robot name="simple_arm" xmlns:xacro="http://www.ros.org/wiki/xacro">
   <xacro:arg name="ros2_control_params" default=""/>
-  <xacro:property name="ros2_control_params" value="$(arg ros2_control_params)"/>
   <material name="gray">
     <color rgba="0.6 0.6 0.6 1.0"/>
@@ -398,5 +397,5 @@
   <gazebo>
     <plugin name="gazebo_ros2_control" filename="libgazebo_ros2_control.so">
-      <parameters>${ros2_control_params}</parameters>
+      <parameters>$(arg ros2_control_params)</parameters>
     </plugin>
   </gazebo>

Commit message: Fix MoveIt2 params and action-based task

File: robot_arm_pick_place/colcon_ws/src/arm_description/urdf/arm.urdf.xacro (robot description, xacro)
@@ -214,5 +214,5 @@
     <origin xyz="0 0 0.025" rpy="0 0 0"/>
     <axis xyz="0 0 1"/>
-    <limit lower="-${pi}" upper="${pi}" effort="50" velocity="1.5"/>
+    <limit lower="-3.141592653589793" upper="3.141592653589793" effort="50" velocity="1.5"/>
   </joint>
   <joint name="joint2" type="revolute">
@@ -221,5 +221,5 @@
     <origin xyz="0 0 0.2" rpy="0 0 0"/>
     <axis xyz="0 1 0"/>
-    <limit lower="-${pi}/2" upper="${pi}/2" effort="50" velocity="1.5"/>
+    <limit lower="-1.57079632679" upper="1.57079632679" effort="50" velocity="1.5"/>
   </joint>
   <joint name="joint3" type="revolute">
@@ -228,5 +228,5 @@
     <origin xyz="0 0 0.25" rpy="0 0 0"/>
     <axis xyz="0 1 0"/>
-    <limit lower="-${pi}/2" upper="${pi}/2" effort="40" velocity="1.5"/>
+    <limit lower="-1.57079632679" upper="1.57079632679" effort="40" velocity="1.5"/>
   </joint>
   <joint name="joint4" type="revolute">
@@ -235,5 +235,5 @@
     <origin xyz="0 0 0.25" rpy="0 0 0"/>
     <axis xyz="1 0 0"/>
-    <limit lower="-${pi}" upper="${pi}" effort="30" velocity="2.0"/>
+    <limit lower="-3.141592653589793" upper="3.141592653589793" effort="30" velocity="2.0"/>
   </joint>
   <joint name="joint5" type="revolute">
@@ -242,5 +242,5 @@
     <origin xyz="0 0 0.2" rpy="0 0 0"/>
     <axis xyz="0 1 0"/>
-    <limit lower="-${pi}" upper="${pi}" effort="20" velocity="2.0"/>
+    <limit lower="-3.141592653589793" upper="3.141592653589793" effort="20" velocity="2.0"/>
   </joint>
   <joint name="joint6" type="revolute">
@@ -249,5 +249,5 @@
     <origin xyz="0 0 0.18" rpy="0 0 0"/>
     <axis xyz="1 0 0"/>
-    <limit lower="-${pi}" upper="${pi}" effort="15" velocity="2.5"/>
+    <limit lower="-3.141592653589793" upper="3.141592653589793" effort="15" velocity="2.5"/>
   </joint>
   <joint name="ee_joint" type="fixed">

Commit message: Add tool0 link and update SRDF tip

File: robot_arm_pick_place/colcon_ws/src/arm_description/urdf/arm.urdf.xacro (robot description, xacro)
@@ -169,4 +169,12 @@
     </inertial>
   </link>
+  <link name="tool0">
+    <visual>
+      <geometry>
+        <sphere radius="0.01"/>
+      </geometry>
+      <material name="red"/>
+    </visual>
+  </link>
   <link name="finger_left">
     <visual>
@@ -256,4 +264,9 @@
     <origin xyz="0 0 0.12" rpy="0 0 0"/>
   </joint>
+  <joint name="tool0_joint" type="fixed">
+    <parent link="ee_link"/>
+    <child link="tool0"/>
+    <origin xyz="0 0 0.05" rpy="0 0 0"/>
+  </joint>
   <joint name="finger_left_joint" type="prismatic">
     <parent link="ee_link"/>

Commit message: Add world fixed joint to anchor base_link

File: robot_arm_pick_place/colcon_ws/src/arm_description/urdf/arm.urdf.xacro (robot description, xacro)
@@ -2,4 +2,10 @@
 <robot name="simple_arm" xmlns:xacro="http://www.ros.org/wiki/xacro">
   <xacro:arg name="ros2_control_params" default=""/>
+  <link name="world"/>
+  <joint name="world_joint" type="fixed">
+    <parent link="world"/>
+    <child link="base_link"/>
+    <origin xyz="0 0 0" rpy="0 0 0"/>
+  </joint>
   <material name="gray">
     <color rgba="0.6 0.6 0.6 1.0"/>

Commit message: Remove base_link inertia for fixed base

File: robot_arm_pick_place/colcon_ws/src/arm_description/urdf/arm.urdf.xacro (robot description, xacro)
@@ -29,9 +29,4 @@
       </geometry>
     </collision>
-    <inertial>
-      <mass value="3.0"/>
-      <origin xyz="0 0 0"/>
-      <inertia ixx="0.01" ixy="0" ixz="0" iyy="0.01" iyz="0" izz="0.01"/>
-    </inertial>
   </link>
   <link name="link1">

Commit message: Add SRDF collision disables and adjust base/table

File: robot_arm_pick_place/colcon_ws/src/arm_description/urdf/arm.urdf.xacro (robot description, xacro)
@@ -22,4 +22,5 @@
         <box size="0.2 0.2 0.05"/>
       </geometry>
+      <origin xyz="0 0 0.025" rpy="0 0 0"/>
       <material name="gray"/>
     </visual>
@@ -28,4 +29,5 @@
         <box size="0.2 0.2 0.05"/>
       </geometry>
+      <origin xyz="0 0 0.025" rpy="0 0 0"/>
     </collision>
   </link>
@@ -221,5 +223,5 @@
     <parent link="base_link"/>
     <child link="link1"/>
-    <origin xyz="0 0 0.025" rpy="0 0 0"/>
+    <origin xyz="0 0 0.05" rpy="0 0 0"/>
     <axis xyz="0 0 1"/>
     <limit lower="-3.141592653589793" upper="3.141592653589793" effort="50" velocity="1.5"/>

Commit message: Remove world link from URDF

File: robot_arm_pick_place/colcon_ws/src/arm_description/urdf/arm.urdf.xacro (robot description, xacro)
@@ -2,10 +2,4 @@
 <robot name="simple_arm" xmlns:xacro="http://www.ros.org/wiki/xacro">
   <xacro:arg name="ros2_control_params" default=""/>
-  <link name="world"/>
-  <joint name="world_joint" type="fixed">
-    <parent link="world"/>
-    <child link="base_link"/>
-    <origin xyz="0 0 0" rpy="0 0 0"/>
-  </joint>
   <material name="gray">
     <color rgba="0.6 0.6 0.6 1.0"/>

Commit message: Restore world joint and remove static TF

File: robot_arm_pick_place/colcon_ws/src/arm_description/urdf/arm.urdf.xacro (robot description, xacro)
@@ -2,4 +2,14 @@
 <robot name="simple_arm" xmlns:xacro="http://www.ros.org/wiki/xacro">
   <xacro:arg name="ros2_control_params" default=""/>
+  <link name="world"/>
+  <joint name="world_joint" type="fixed">
+    <parent link="world"/>
+    <child link="base_link"/>
+    <origin xyz="0 0 0" rpy="0 0 0"/>
+  </joint>
+  <gazebo reference="world_joint">
+    <disableFixedJointLumping>true</disableFixedJointLumping>
+    <preserveFixedJoint>true</preserveFixedJoint>
+  </gazebo>
   <material name="gray">
     <color rgba="0.6 0.6 0.6 1.0"/>
@@ -25,4 +35,9 @@
       <origin xyz="0 0 0.025" rpy="0 0 0"/>
     </collision>
+    <inertial>
+      <mass value="3.0"/>
+      <origin xyz="0 0 0.025"/>
+      <inertia ixx="0.01" ixy="0" ixz="0" iyy="0.01" iyz="0" izz="0.01"/>
+    </inertial>
   </link>
   <link name="link1">

Commit message: Relax gripper lower joint limits

File: robot_arm_pick_place/colcon_ws/src/arm_description/urdf/arm.urdf.xacro (robot description, xacro)
@@ -286,5 +286,5 @@
     <origin xyz="0.03 0.03 0" rpy="0 0 0"/>
     <axis xyz="0 0 1"/>
-    <limit lower="0.0" upper="0.04" effort="10" velocity="0.2"/>
+    <limit lower="-0.001" upper="0.04" effort="10" velocity="0.2"/>
   </joint>
   <joint name="finger_right_joint" type="prismatic">
@@ -293,5 +293,5 @@
     <origin xyz="0.03 -0.03 0" rpy="0 0 0"/>
     <axis xyz="0 0 1"/>
-    <limit lower="0.0" upper="0.04" effort="10" velocity="0.2"/>
+    <limit lower="-0.001" upper="0.04" effort="10" velocity="0.2"/>
   </joint>
   <ros2_control name="ArmSystem" type="system">

Commit message: Load MoveIt configs and relax gripper limits

File: robot_arm_pick_place/colcon_ws/src/arm_description/urdf/arm.urdf.xacro (robot description, xacro)
@@ -286,5 +286,5 @@
     <origin xyz="0.03 0.03 0" rpy="0 0 0"/>
     <axis xyz="0 0 1"/>
-    <limit lower="-0.001" upper="0.04" effort="10" velocity="0.2"/>
+    <limit lower="-0.01" upper="0.04" effort="10" velocity="0.2"/>
   </joint>
   <joint name="finger_right_joint" type="prismatic">
@@ -293,5 +293,5 @@
     <origin xyz="0.03 -0.03 0" rpy="0 0 0"/>
     <axis xyz="0 0 1"/>
-    <limit lower="-0.001" upper="0.04" effort="10" velocity="0.2"/>
+    <limit lower="-0.01" upper="0.04" effort="10" velocity="0.2"/>
   </joint>
   <ros2_control name="ArmSystem" type="system">

Commit message: Fix spin deadlocks and gripper axis

File: robot_arm_pick_place/colcon_ws/src/arm_description/urdf/arm.urdf.xacro (robot description, xacro)
@@ -285,5 +285,5 @@
     <child link="finger_left"/>
     <origin xyz="0.03 0.03 0" rpy="0 0 0"/>
-    <axis xyz="0 0 1"/>
+    <axis xyz="0 1 0"/>
     <limit lower="-0.01" upper="0.04" effort="10" velocity="0.2"/>
   </joint>
@@ -292,5 +292,5 @@
     <child link="finger_right"/>
     <origin xyz="0.03 -0.03 0" rpy="0 0 0"/>
-    <axis xyz="0 0 1"/>
+    <axis xyz="0 -1 0"/>
     <limit lower="-0.01" upper="0.04" effort="10" velocity="0.2"/>
   </joint>

Commit message: Fix gripper axis and adjust grasp height

File: robot_arm_pick_place/colcon_ws/src/arm_description/urdf/arm.urdf.xacro (robot description, xacro)
@@ -284,6 +284,6 @@
     <parent link="ee_link"/>
     <child link="finger_left"/>
-    <origin xyz="0.03 0.03 0" rpy="0 0 0"/>
-    <axis xyz="0 0 1"/>
+    <origin xyz="0.03 0.025 0" rpy="0 0 0"/>
+    <axis xyz="0 1 0"/>
     <limit lower="-0.01" upper="0.04" effort="10" velocity="0.2"/>
   </joint>
@@ -291,6 +291,6 @@
     <parent link="ee_link"/>
     <child link="finger_right"/>
-    <origin xyz="0.03 -0.03 0" rpy="0 0 0"/>
-    <axis xyz="0 0 1"/>
+    <origin xyz="0.03 -0.025 0" rpy="0 0 0"/>
+    <axis xyz="0 -1 0"/>
     <limit lower="-0.01" upper="0.04" effort="10" velocity="0.2"/>
   </joint>

Commit message: Update pick/place pipeline and color cycle behavior

File: robot_arm_pick_place/colcon_ws/src/arm_description/urdf/arm.urdf.xacro (robot description, xacro)
@@ -229,4 +229,18 @@
     </inertial>
   </link>
+  <link name="camera_link">
+    <visual>
+      <geometry>
+        <box size="0.03 0.03 0.02"/>
+      </geometry>
+      <origin xyz="0 0 0.01" rpy="0 0 0"/>
+      <material name="gray"/>
+    </visual>
+    <inertial>
+      <mass value="0.05"/>
+      <origin xyz="0 0 0.01"/>
+      <inertia ixx="0.0001" ixy="0" ixz="0" iyy="0.0001" iyz="0" izz="0.0001"/>
+    </inertial>
+  </link>
   <joint name="joint1" type="revolute">
     <parent link="base_link"/>
@@ -295,4 +309,36 @@
     <limit lower="-0.01" upper="0.04" effort="10" velocity="0.2"/>
   </joint>
+  <joint name="camera_joint" type="fixed">
+    <parent link="ee_link"/>
+    <child link="camera_link"/>
+    <origin xyz="0.12 0.0 0.08" rpy="0 -0.6 0"/>
+  </joint>
+  <gazebo reference="camera_link">
+    <sensor name="camera" type="camera">
+      <update_rate>30</update_rate>
+      <camera>
+        <horizontal_fov>0.8</horizontal_fov>
+        <image>
+          <width>640</width>
+          <height>480</height>
+          <format>R8G8B8</format>
+        </image>
+        <clip>
+          <near>0.05</near>
+          <far>10.0</far>
+        </clip>
+      </camera>
+      <plugin name="gazebo_ros_camera" filename="libgazebo_ros_camera.so">
+        <ros>
+          <namespace>/camera</namespace>
+        </ros>
+        <camera_name>color</camera_name>
+        <image_topic_name>image_raw</image_topic_name>
+        <camera_info_topic_name>camera_info</camera_info_topic_name>
+        <frame_name>camera_link</frame_name>
+      </plugin>
+    </sensor>
+  </gazebo>
+  <!-- Overhead camera sensors are defined in the Gazebo world for stable pose control. -->
   <ros2_control name="ArmSystem" type="system">
     <hardware>
